File: H1FR10/Design/H1FR10.brd (EAGLE design)
At the start: 34.6 x 30 mm, 22 parts, among them J1 U.FL-R-SMT-1_10_, P1 HEXABIT_17.32_NO_P6_P7_P12, U1 STM32G0B1CEU6N, U2 LORA127X-C1, X1 XTALL_CSTCE8M00G52

Commit message: -Correct some documentaion issues
Parts:
- U2: value LORA127X-C1 -> Lora1276-C1-868
Changed lines of the file:
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@@
 <drawing>
 <settings>
-<setting alwaysvectorfont="yes"/>
+<setting alwaysvectorfont="no"/>
 <setting verticaltext="up"/>
 </settings>
@@
 </layers>
 <board>
-<fusionsync huburn="a.YnVzaW5lc3M6Z21haWwyMzYzMzA4" projecturn="a.YnVzaW5lc3M6Z21haWwyMzYzMzA4I0QyMDIyMDIyNzUwMTk3Njc4MQ" f3durn="urn:adsk.wipprod:dm.lineage:g33QiWTATBWUxJrgd01D7A" pcbguid="a9d9cf8e-6004-470c-9fae-bded3e58f8ae" lastpulledtime="" lastsyncedchangeguid="" latestrevisionid="963eccc5-135f-44c9-b6fb-1757420cdf18" lastsyncedrevisionid="963eccc5-135f-44c9-b6fb-1757420cdf18" lastboardhashguid="916340fe-12a8-a5dc-f2dd-82a76867899b" lastpushedtime="2023-11-14T15:43:17Z" linktopcb3d="true"/>
+<fusionsync huburn="a.YnVzaW5lc3M6Z21haWwyMzYzMzA4" projecturn="a.YnVzaW5lc3M6Z21haWwyMzYzMzA4I0QyMDIyMDIyNzUwMTk3Njc4MQ" f3durn="urn:adsk.wipprod:dm.lineage:g33QiWTATBWUxJrgd01D7A" pcbguid="" lastpulledtime="" lastsyncedchangeguid="" latestrevisionid="963eccc5-135f-44c9-b6fb-1757420cdf18" lastsyncedrevisionid="963eccc5-135f-44c9-b6fb-1757420cdf18" lastboardhashguid="916340fe-12a8-a5dc-f2dd-82a76867899b" lastpushedtime="2023-11-14T15:43:17Z" linktopcb3d="true"/>
 <plain>
 <rectangle x1="-6.400928125" y1="5.00976875" x2="-5.649596875" y2="5.0245" layer="21"/>
@@
 </element>
 <element name="P1" library="hexabitz_connectors" library_urn="urn:adsk.eagle:library:20064578" package="HEXABIT_17.32_NO_P6_P7_P12" package3d_urn="urn:adsk.eagle:package:20064634/2" value="HEXABIT_17.32_NO_P6_P7_P12" x="0" y="15.08125" smashed="yes"/>
-<element name="U2" library="HEXABITZ_ICs" library_urn="urn:adsk.eagle:library:20064554" package="LORA127X-C1" package3d_urn="urn:adsk.eagle:package:42421660/4" value="LORA127X-C1" x="0.15875" y="17.62125" smashed="yes" rot="R180">
+<element name="U2" library="HEXABITZ_ICs" library_urn="urn:adsk.eagle:library:20064554" package="LORA127X-C1" package3d_urn="urn:adsk.eagle:package:42421660/4" value="Lora1276-C1-868" x="0.15875" y="17.62125" smashed="yes" rot="R180">
 <attribute name="AVAILABILITY" value="Not in stock" x="0.15875" y="17.62125" size="1.778" layer="27" rot="R180" display="off"/>
 <attribute name="CHECK_PRICES" value="https://www.snapeda.com/parts/ESP8266-12E/ESP-12E/AI-Thinker/view-part/?ref=eda" x="0.15875" y="17.62125" size="1.778" layer="27" rot="R180" display="off"/>
